File: board/board.kicad_sch (KiCad schematic)
At the start: 10 parts, among them Q1 2N7002, U1 ATtiny402-SS

Commit message: fixed schematic and pcb
Parts:
- removed Q1: 2N7002, Package_TO_SOT_SMD:SOT-23, symbol Transistor_FET:2N7002
- added C3: 10u, Capacitor_SMD:C_0603_1608Metric_Pad1.08x0.95mm_HandSolder, symbol Device:C
- added Q1: AO3401A, Package_TO_SOT_SMD:SOT-23, symbol Transistor_FET:AO3401A
- added TP1: TestPoint, TestPoint:TestPoint_Pad_D1.0mm, symbol Connector:TestPoint
Connections:
- net GND_BT is gone; now on net GND: C2.2
- net +4V: now also R2.2, C3.1, Q1.2 (S); no longer U3.1 (Vcc)
- net GND: now also C3.2; no longer R2.1
- net UPDI: now also TP1.1; no longer U3.3 (UPDI)
- net at R1.1: now also R2.1, Q1.1 (G); no longer R2.2
- net IO_SCAN: now reaches U1.2 (PA6)
- net IO_SCAN: now also U3.3 (SCAN)
- new net Vcc_BT: Q1.3 (D), U3.1 (VCC_BT)
- no-connect marks 1 -> 0
Other:
- moved on the sheet: C2, R2
